Commit message: Added urdfviewer

File: URDF/Complete Arm Assembly/urdf/Complete Arm Assembly.urdf (robot description, URDF)
Before this commit: robot Complete Arm Assembly, 8 links, 5 joints
Joints:
- removed joint joint_5
- added joint left_finger_joint: type revolute, parent end_effector, child left_finger, origin xyz=1.5222 -1.1548 -0.7061 rpy=-1.5708 -1.5708 0, axis 0 1 0, limit lower=0.0 upper=0.019 effort=0.5 velocity=0.5, mimic joint=right_finger_joint multiplier=-1 offset=0
- added joint right_finger_joint: type revolute, parent end_effector, child right_finger, origin xyz=1.5222 -1.0976 -0.7061 rpy=-1.5708 -1.5708 0, axis 0 1 0, limit lower=0.0 upper=0.019 effort=0.5 velocity=0.5
- added joint wrist_rotate_joint: type revolute, parent link_4, child end_effector, origin xyz=0.2223 0.24575 0.0005 rpy=0 1.5708 0, axis 0 0 1, limit lower=-3.14159 upper=3.14159 effort=1.0 velocity=1.0
- joint joint_1: limit lower=0 upper=0 effort=0 velocity=0 -> lower=-3.14159 upper=3.14159 effort=1.0 velocity=1.0
- joint joint_2: axis 0 0 0 -> 0 1 0; limit lower=0 upper=0 effort=0 velocity=0 -> lower=-1.5708 upper=1.5708 effort=1.0 velocity=1.0
- joint joint_3: axis 0 0 0 -> 0 1 0; limit lower=0 upper=0 effort=0 velocity=0 -> lower=-1.5708 upper=1.5708 effort=1.0 velocity=1.0
- joint joint_4: axis 0 0 0 -> 0 1 0; limit lower=0 upper=0 effort=0 velocity=0 -> lower=-1.5708 upper=1.5708 effort=1.0 velocity=1.0
