Commit message: Added the updated URDF file

File: URDF/complete_arm_assembly/urdf/Complete Arm Assembly.urdf (robot description, URDF)
Before this commit: robot Complete_Arm_Assembly, 8 links, 7 joints
Links:
- link base_link: mass 0.0944596926666318 -> 0.0426185203491502
- link end_effector: mass 0.0448261455614491 -> 0.0448261455614486
- link left_finger: mass 0.0287713290324178 -> 0.028771329032418
- link link_1: mass 0.04515255146413 -> 0.0451525514641292
- link link_2: mass 0.0676816456886685 -> 0.067681645688669
- link link_3: mass 0.0616267578939111 -> 0.0616267578939116
- link right_finger: mass 0.0287713290324161 -> 0.0287713290324179
Joints:
- removed joint wrist_rotate_joint
- added joint joint_5: type revolute, parent link_4, child end_effector, origin xyz=0.2223 0.24575 0.0005 rpy=0 1.5708 0, axis 1 0 0, limit lower=0 upper=0 effort=0 velocity=0
- joint joint_1: limit lower=-3.14159 upper=3.14159 effort=1.0 velocity=1.0 -> lower=0 upper=0 effort=0 velocity=0
- joint joint_2: axis 0 1 0 -> 0 0 1; limit lower=-1.5708 upper=1.5708 effort=1.0 velocity=1.0 -> lower=0 upper=0 effort=0 velocity=0
- joint joint_3: axis 0 1 0 -> 0 0 1; limit lower=-1.5708 upper=1.5708 effort=1.0 velocity=1.0 -> lower=0 upper=0 effort=0 velocity=0
- joint joint_4: axis 0 1 0 -> 0 0 1; limit lower=-1.5708 upper=1.5708 effort=1.0 velocity=1.0 -> lower=0 upper=0 effort=0 velocity=0
- joint left_finger_joint: axis 0 1 0 -> 1 0 0; limit lower=0.0 upper=0.019 effort=0.5 velocity=0.5 -> lower=0 upper=0 effort=0 velocity=0; origin xyz=1.5222 -1.1548 -0.7061 rpy=-1.5708 -1.5708 0 -> xyz=1.3371 -1.1093 -0.83538 rpy=3.1416 -1.5708 0; type revolute -> prismatic
- joint right_finger_joint: axis 0 1 0 -> 1 0 0; limit lower=0.0 upper=0.019 effort=0.5 velocity=0.5 -> lower=0 upper=0 effort=0 velocity=0; origin xyz=1.5222 -1.0976 -0.7061 rpy=-1.5708 -1.5708 0 -> xyz=1.2858 -1.1091 -0.83518 rpy=3.1416 -1.5708 0; type revolute -> prismatic
