Commit message: Fixed the xacro file to have the correct z-position for fingers

File: URDF/complete_arm_assembly/urdf/Complete Arm Assembly.urdf.xacro (robot description, xacro)
@@ -4,5 +4,17 @@
      For more information, please see http://wiki.ros.org/sw_urdf_exporter -->
 <robot
-  name="Complete Arm Assembly">
+  name="Complete Arm Assembly"
+  xmlns:xacro="http://www.ros.org/wiki/xacro">
+  <!-- ===== Finger joint position properties ===== -->
+  <!-- z offset relative to end_effector frame: world_finger_z - ee_world_z = 0 -->
+  <xacro:property name="ee_world_z"     value="0.0005"/>  <!-- from joint_5 z -->
+  <xacro:property name="world_finger_z" value="0.0005"/>  <!-- fingers sit at same z as end_effector -->
+  <xacro:property name="finger_local_z" value="${world_finger_z - ee_world_z}"/>
+  <!-- Right finger x/y offsets (unchanged) -->
+  <xacro:property name="rf_x" value="1.2858"/>
+  <xacro:property name="rf_y" value="-1.1091"/>
+  <!-- Left finger x/y offsets (unchanged) -->
+  <xacro:property name="lf_x" value="1.3371"/>
+  <xacro:property name="lf_y" value="-1.1093"/>
   <link
     name="base_link">
@@ -379,5 +391,5 @@
     type="prismatic">
     <origin
-      xyz="1.2858 -1.1091 -0.83518"
+      xyz="${rf_x} ${rf_y} ${finger_local_z}"
       rpy="3.1416 -1.5708 0" />
     <parent
@@ -437,5 +449,5 @@
     type="prismatic">
     <origin
-      xyz="1.3371 -1.1093 -0.83538"
+      xyz="${lf_x} ${lf_y} ${finger_local_z}"
       rpy="3.1416 -1.5708 0" />
     <parent
