Commit message: Updated the file from Solidworks

File: complete_arm_assembly/urdf/complete_arm_assembly.urdf (robot description, URDF)
Before this commit: robot Complete Arm Assembly, 8 links, 7 joints
Links:
- removed link end_effector
- added link link_5, mass 0.085015418080232; collision mesh filename=package://complete_arm_assembly/meshes/link_5.STL; visual mesh filename=package://complete_arm_assembly/meshes/link_5.STL
- link base_link: mass 0.0426185203491502 -> 0.0944596926666338; geometry collision mesh filename=package://complete_arm_assembly/meshes/base_link.STL; visual mesh filename=package://complete_arm_assembly/meshes/base_link.STL
- link left_finger: mass 0.028771329032418 -> 0.0274218714255595; geometry collision mesh filename=package://complete_arm_assembly/meshes/left_finger.STL; visual mesh filename=package://complete_arm_assembly/meshes/left_finger.STL
- link link_1: mass 0.0451525514641292 -> 0.0446962058831376; geometry collision mesh filename=package://complete_arm_assembly/meshes/link_1.STL; visual mesh filename=package://complete_arm_assembly/meshes/link_1.STL
- link link_2: mass 0.067681645688669 -> 0.0672253268158646; geometry collision mesh filename=package://complete_arm_assembly/meshes/link_2.STL; visual mesh filename=package://complete_arm_assembly/meshes/link_2.STL
- link link_3: mass 0.0616267578939116 -> 0.0611704285828677; geometry collision mesh filename=package://complete_arm_assembly/meshes/link_3.STL; visual mesh filename=package://complete_arm_assembly/meshes/link_3.STL
- link link_4: mass 0.181115636338247 -> 0.181115636310511; geometry collision mesh filename=package://complete_arm_assembly/meshes/link_4.STL; visual mesh filename=package://complete_arm_assembly/meshes/link_4.STL
- link right_finger: mass 0.0287713290324179 -> 0.0274218653592185; geometry collision mesh filename=package://complete_arm_assembly/meshes/right_finger.STL; visual mesh filename=package://complete_arm_assembly/meshes/right_finger.STL
Joints:
- removed joint joint_2
- added joint joint)2: type revolute, parent link_1, child link_2, origin xyz=0 0.040505 0 rpy=0 0 0.75692, axis 0 0 1, limit lower=0 upper=0 effort=0 velocity=0
- joint joint_1: origin xyz=0.69033 -1.3112 0.92243 rpy=1.5708 0 0 -> xyz=-0.00078087 -1.0373 0.041025 rpy=1.5708 0 0.52968
- joint joint_3: origin xyz=-0.0585 0.2105 0 rpy=3.1416 0 1.5708 -> xyz=0.024 0.128 0 rpy=0 0 0.23095
- joint joint_4: origin xyz=-0.2105 0.0585 0 rpy=3.1416 0 1.5708 -> xyz=0.124 0 0 rpy=0 0 -0.98787
- joint joint_5: child end_effector -> link_5; origin xyz=0.2223 0.24575 0.0005 rpy=0 1.5708 0 -> xyz=0.086402 0.02425 0.0005 rpy=0.036324 0 0
- joint left_finger_joint: mimic joint=right_finger_joint multiplier=-1 offset=0 -> (none); origin xyz=${lf_x} ${lf_y} ${finger_local_z} rpy=3.1416 -1.5708 0 -> xyz=-0.019263 -1.6285 -1.7856 rpy=0 0 0; parent end_effector -> link_5
- joint right_finger_joint: mimic (none) -> joint=left_finger_joint multiplier=-1 offset=0; origin xyz=${rf_x} ${rf_y} ${finger_local_z} rpy=3.1416 -1.5708 0 -> xyz=0.099706 -1.7393 -1.982 rpy=0 0 0; parent end_effector -> link_5

Commit message: Updated the right finger postion

File: complete_arm_assembly/urdf/complete_arm_assembly.urdf (robot description, URDF)
Before this commit: robot complete_arm_assembly, 8 links, 7 joints
Links:
- link left_finger: mass 0.0274218714255595 -> 0.0274218702393672
- link link_2: mass 0.0672253268158646 -> 0.0672255298525689
- link link_3: mass 0.0611704285828677 -> 0.0611704168846414
- link link_5: mass 0.085015418080232 -> 0.0850149357001051
- link right_finger: mass 0.0274218653592185 -> 0.0274218628103089
Joints:
- joint joint)2: origin xyz=0 0.040505 0 rpy=0 0 0.75692 -> xyz=0 0.0405050009999363 0 rpy=0 0 0.75692376857971
- joint joint_1: origin xyz=-0.00078087 -1.0373 0.041025 rpy=1.5708 0 0.52968 -> xyz=-0.000780869923727945 -1.0372656750587 0.0410248897442467 rpy=1.5707963267949 0 0.52968486830993
- joint joint_3: origin xyz=0.024 0.128 0 rpy=0 0 0.23095 -> xyz=0.0240000000000004 0.128 0 rpy=0 0 0.230949108410148
- joint joint_4: origin xyz=0.124 0 0 rpy=0 0 -0.98787 -> xyz=0.123999999999999 0 0 rpy=0 0 -0.987872876989858
- joint joint_5: origin xyz=0.086402 0.02425 0.0005 rpy=0.036324 0 0 -> xyz=0.0864019800647668 0.0242500000276551 0.000500000021411151 rpy=0.036323657737331 0 0
- joint right_finger_joint: origin xyz=0.099706 -1.7393 -1.982 rpy=0 0 0 -> xyz=0.12146 -0.020109 -2.6376 rpy=0 0 0

Commit message: Adjusted right finger postion

File: complete_arm_assembly/urdf/complete_arm_assembly.urdf (robot description, URDF)
Before this commit: robot complete_arm_assembly, 8 links, 7 joints
Joints:
- joint right_finger_joint: axis 1 0 0 -> 0 0 0; origin xyz=0.12146 -0.020109 -2.6376 rpy=0 0 0 -> xyz=0.12146 -0.020109 -2.6376 rpy=0.69955 0 0

Commit message: Adjusted right finger postion

File: complete_arm_assembly/urdf/complete_arm_assembly.urdf (robot description, URDF)
Before this commit: robot complete_arm_assembly, 8 links, 7 joints
Links:
- link right_finger: mass 0.0274218628103089 -> 0.0274218628103051
Joints:
- removed joint joint)2
- added joint joint_2: type revolute, parent link_1, child link_2, origin xyz=0 0.040505 0 rpy=0 0 0.31732, axis 0 0 1, limit lower=0 upper=0 effort=0 velocity=0
- joint joint_1: origin xyz=-0.000780869923727945 -1.0372656750587 0.0410248897442467 rpy=1.5707963267949 0 0.52968486830993 -> xyz=-0.00078087 -1.0373 0.041025 rpy=1.5708 0 0.52968
- joint joint_3: origin xyz=0.0240000000000004 0.128 0 rpy=0 0 0.230949108410148 -> xyz=0.024 0.128 0 rpy=0 0 0.95298
- joint joint_4: origin xyz=0.123999999999999 0 0 rpy=0 0 -0.987872876989858 -> xyz=0.124 0 0 rpy=0 0 -1.2703
- joint joint_5: origin xyz=0.0864019800647668 0.0242500000276551 0.000500000021411151 rpy=0.036323657737331 0 0 -> xyz=0.086402 0.02425 0.0005 rpy=0.73588 0 0
- joint right_finger_joint: axis 0 0 0 -> 1 0 0; origin xyz=0.12146 -0.020109 -2.6376 rpy=0.69955 0 0 -> xyz=-0.019263 1.6058 1.7856 rpy=-3.1416 0 0

Commit message: Fixed the positioning

File: complete_arm_assembly/urdf/complete_arm_assembly.urdf (robot description, URDF)
Before this commit: robot complete_arm_assembly, 8 links, 7 joints
Links:
- added link world
- link base_link: geometry collision mesh filename=file:///home/ri-one/Open-Manipulator-X-6/complete_arm_assem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; visual mesh filename=file:///home/ri-one/Open-Manipulator-X-6/complete_arm_assem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
- link left_finger: mass 0.0274218702393672 -> 0.0274218714255595; geometry collision mesh filename=file:///home/ri-one/Open-Manipulator-X-6/complete_arm_assem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; visual mesh filename=file:///home/ri-one/Open-Manipulator-X-6/complete_arm_assem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
- link link_1: geometry collision mesh filename=file:///home/ri-one/Open-Manipulator-X-6/complete_arm_assem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; visual mesh filename=file:///home/ri-one/Open-Manipulator-X-6/complete_arm_assem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
- link link_2: mass 0.0672255298525689 -> 0.0672253268158646; geometry collision mesh filename=file:///home/ri-one/Open-Manipulator-X-6/complete_arm_assem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; visual mesh filename=file:///home/ri-one/Open-Manipulator-X-6/complete_arm_assem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
- link link_3: mass 0.0611704168846414 -> 0.0611704285828677; geometry collision mesh filename=file:///home/ri-one/Open-Manipulator-X-6/complete_arm_assem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; visual mesh filename=file:///home/ri-one/Open-Manipulator-X-6/complete_arm_assem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
- link link_4: geometry collision mesh filename=file:///home/ri-one/Open-Manipulator-X-6/complete_arm_assem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; visual mesh filename=file:///home/ri-one/Open-Manipulator-X-6/complete_arm_assem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
- link link_5: mass 0.0850149357001051 -> 0.085015418080232; geometry collision mesh filename=file:///home/ri-one/Open-Manipulator-X-6/complete_arm_assem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; visual mesh filename=file:///home/ri-one/Open-Manipulator-X-6/complete_arm_assem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
- link right_finger: mass 0.0274218628103051 -> 0.0274218653592185; geometry collision mesh filename=file:///home/ri-one/Open-Manipulator-X-6/complete_arm_assem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; visual mesh filename=file:///home/ri-one/Open-Manipulator-X-6/complete_arm_assem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
Joints:
- added joint world_to_base_joint: type fixed, parent world, child base_link, origin xyz=0 0 0 rpy=0 0 0
- joint joint_1: limit lower=0 upper=0 effort=0 velocity=0 -> lower=-3.14 upper=3.14 effort=10 velocity=1
- joint joint_2: limit lower=0 upper=0 effort=0 velocity=0 -> lower=-1.57 upper=1.57 effort=10 velocity=1; origin xyz=0 0.040505 0 rpy=0 0 0.31732 -> xyz=0 0.040505 0 rpy=0 0 0.75692
- joint joint_3: limit lower=0 upper=0 effort=0 velocity=0 -> lower=-1.57 upper=1.57 effort=10 velocity=1; origin xyz=0.024 0.128 0 rpy=0 0 0.95298 -> xyz=0.024 0.128 0 rpy=0 0 0.23095
- joint joint_4: limit lower=0 upper=0 effort=0 velocity=0 -> lower=-1 upper=2. effort=10 velocity=1; origin xyz=0.124 0 0 rpy=0 0 -1.2703 -> xyz=0.124 0 0 rpy=0 0 -0.98787
- joint joint_5: limit lower=0 upper=0 effort=0 velocity=0 -> lower=-3.14 upper=3.14 effort=10 velocity=1; origin xyz=0.086402 0.02425 0.0005 rpy=0.73588 0 0 -> xyz=0.086402 0.02425 0.0005 rpy=0.036324 0 0
- joint left_finger_joint: axis 1 0 0 -> 0 0 1; limit lower=0 upper=0 effort=0 velocity=0 -> lower=0 upper=0.019 effort=5 velocity=0.1
- joint right_finger_joint: axis 1 0 0 -> 0 0 -1

File: complete_arm_assembly/urdf/complete_arm_assembly_urdf.xacro (robot description, xacro)
@@ -1,458 +1,274 @@
 <?xml version="1.0" encoding="utf-8"?>
-<!-- This URDF was automatically created by SolidWorks to URDF Exporter! Originally created by Stephen Brawner (brawner@gmail.com)
-     Commit Version: 1.6.0-4-g7f85cfe  Build Version: 1.6.7995.38578
-     For more information, please see http://wiki.ros.org/sw_urdf_exporter -->
-<robot
-  name="complete_arm_assembly">
-  <link
-    name="base_link">
-    <inertial>
-      <origin
-        xyz="-0.0126522064234279 0.0112081741589456 1.03738375057827"
-        rpy="0 0 0" />
-      <mass
-        value="0.0944596926666338" />
-      <inertia
-        ixx="2.49395953752317E-05"
-        ixy="-1.07943571271723E-07"
-        ixz="1.09620010475091E-09"
-        iyy="4.59171379732495E-05"
-        iyz="8.47831697329351E-09"
-        izz="3.13098479474975E-05" />
-    </inertial>
-    <visual>
-      <origin
-        xyz="0 0 0"
-        rpy="0 0 0" />
-      <geometry>
-        <mesh
-          filename="file:///home/ri-one/Open-Manipulator-X-6/complete_arm_assembly/urdf/../meshes/base_link.STL" />
-      </geometry>
-      <material
-        name="">
-        <color
-          rgba="0.894117647058823 0.894117647058823 0.894117647058823 1" />
-      </material>
-    </visual>
-    <collision>
-      <origin
-        xyz="0 0 0"
-        rpy="0 0 0" />
-      <geometry>
-        <mesh
-          filename="file:///home/ri-one/Open-Manipulator-X-6/complete_arm_assembly/urdf/../meshes/base_link.STL" />
-      </geometry>
-    </collision>
-  </link>
-  <link
-    name="link_1">
-    <inertial>
-      <origin
-        xyz="-1.21952357101662E-08 0.0275827025842473 0.000932155095934251"
-        rpy="0 0 0" />
-      <mass
-        value="0.0446962058831376" />
-      <inertia
-        ixx="1.2281031278665E-05"
-        ixy="1.20613706130026E-12"
-        ixz="7.89362412536608E-12"
-        iyy="7.29718852707007E-06"
-        iyz="-1.08328965106875E-07"
-        izz="1.06262085935607E-05" />
-    </inertial>
-    <visual>
-      <origin
-        xyz="0 0 0"
-        rpy="0 0 0" />
-      <geometry>
-        <mesh
-          filename="file:///home/ri-one/Open-Manipulator-X-6/complete_arm_assembly/urdf/../meshes/link_1.STL" />
-      </geometry>
-      <material
-        name="">
-        <color
-          rgba="0.894117647058823 0.894117647058823 0.894117647058823 1" />
-      </material>
-    </visual>
-    <collision>
-      <origin
-        xyz="0 0 0"
-        rpy="0 0 0" />
-      <geometry>
-        <mesh
-          filename="file:///home/ri-one/Open-Manipulator-X-6/complete_arm_assembly/urdf/../meshes/link_1.STL" />
-      </geometry>
-    </collision>
-  </link>
-  <joint
-    name="joint_1"
-    type="revolute">
-    <origin
-      xyz="-0.00078087 -1.0373 0.041025"
-      rpy="1.5708 0 0.52968" />
-    <parent
-      link="base_link" />
-    <child
-      link="link_1" />
-    <axis
-      xyz="0 1 0" />
-    <limit
-      lower="-3.14"
-      upper="3.14"
-      effort="10"
-      velocity="1" />
-  </joint>
-  <link
-    name="link_2">
-    <inertial>
-      <origin
-        xyz="0.0083495112245085 0.104913808310048 0.00061978124354245"
-        rpy="0 0 0" />
-      <mass
-        value="0.0672253268158646" />
-      <inertia
-        ixx="2.05051000460793E-05"
-        ixy="3.5213726037406E-11"
-        ixz="-1.08338604683114E-07"
-        iyy="1.6315288025526E-05"
-        iyz="-1.50521736891554E-11"
-        izz="2.2628963418613E-05" />
-    </inertial>
-    <visual>
-      <origin
-        xyz="0 0 0"
-        rpy="0 0 0" />
-      <geometry>
-        <mesh
-          filename="file:///home/ri-one/Open-Manipulator-X-6/complete_arm_assembly/urdf/../meshes/link_2.STL" />
-      </geometry>
-      <material
-        name="">
-        <color
-          rgba="0.894117647058823 0.894117647058823 0.894117647058823 1" />
-      </material>
-    </visual>
-    <collision>
-      <origin
-        xyz="0 0 0"
-        rpy="0 0 0" />
-      <geometry>
-        <mesh
-          filename="file:///home/ri-one/Open-Manipulator-X-6/complete_arm_assembly/urdf/../meshes/link_2.STL" />
-      </geometry>
-    </collision>
-  </link>
-  <joint
-    name="joint)2"
-    type="revolute">
-    <origin
-      xyz="0 0.040505 0"
-      rpy="0 0 0.75692" />
-    <parent
-      link="link_1" />
-    <child
-      link="link_2" />
-    <axis
-      xyz="0 0 1" />
-    <limit
-      lower="-1.57"
-      upper="1.57"
-      effort="10"
-      velocity="1" />
-  </joint>
-  <link
-    name="link_3">
-    <inertial>
-      <origin
-        xyz="0.0935866065506837 6.68493950972682E-07 0.000681111440057891"
-        rpy="0 0 0" />
-      <mass
-        value="0.0611704285828677" />
-      <inertia
-        ixx="1.00859846466543E-05"
-        ixy="-2.12087916751726E-11"
-        ixz="-1.08328219187182E-07"
-        iyy="1.83430482645789E-05"
-        iyz="-8.84540758950517E-12"
-        izz="1.53128572066901E-05" />
-    </inertial>
-    <visual>
-      <origin
-        xyz="0 0 0"
-        rpy="0 0 0" />
-      <geometry>
-        <mesh
-          filename="file:///home/ri-one/Open-Manipulator-X-6/complete_arm_assembly/urdf/../meshes/link_3.STL" />
-      </geometry>
-      <material
-        name="">
-        <color
-          rgba="0.894117647058823 0.894117647058823 0.894117647058823 1" />
-      </material>
-    </visual>
-    <collision>
-      <origin
-        xyz="0 0 0"
-        rpy="0 0 0" />
-      <geometry>
-        <mesh
-          filename="file:///home/ri-one/Open-Manipulator-X-6/complete_arm_assembly/urdf/../meshes/link_3.STL" />
-      </geometry>
-    </collision>
-  </link>
-  <joint
-    name="joint_3"
-    type="revolute">
-    <origin
-      xyz="0.024 0.128 0"
-      rpy="0 0 0.23095" />
-    <parent
-      link="link_2" />
-    <child
-      link="link_3" />
-    <axis
-      xyz="0 0 1" />
-    <limit
-      lower="-1.57"
-      upper="1.57"
-      effort="10"
-      velocity="1" />
-  </joint>
-  <link
-    name="link_4">
-    <inertial>
-      <origin
-        xyz="0.050731760745883 0.011797475505387 -0.000207275711230026"
-        rpy="0 0 0" />
-      <mass
-        value="0.181115636310511" />
-      <inertia
-        ixx="0.000125082991142915"
-        ixy="-1.91715165837534E-07"
-        ixz="-3.18809483889817E-07"
-        iyy="7.52710719120373E-05"
-        iyz="2.8145647428354E-09"
-        izz="7.57487395968248E-05" />
-    </inertial>
-    <visual>
-      <origin
-        xyz="0 0 0"
-        rpy="0 0 0" />
-      <geometry>
-        <mesh
-          filename="file:///home/ri-one/Open-Manipulator-X-6/complete_arm_assembly/urdf/../meshes/link_4.STL" />
-      </geometry>
-      <material
-        name="">
-        <color
-          rgba="0.894117647058823 0.894117647058823 0.894117647058823 1" />
-      </material>
-    </visual>
-    <collision>
-      <origin
-        xyz="0 0 0"
-        rpy="0 0 0" />
-      <geometry>
-        <mesh
-          filename="file:///home/ri-one/Open-Manipulator-X-6/complete_arm_assembly/urdf/../meshes/link_4.STL" />
-      </geometry>
-    </collision>
-  </link>
-  <joint
-    name="joint_4"
-    type="revolute">
-    <origin
-      xyz="0.124 0 0"
-      rpy="0 0 -0.98787" />
-    <parent
-      link="link_3" />
-    <child
-      link="link_4" />
-    <axis
-      xyz="0 0 1" />
-    <limit
-      lower="-1"
-      upper="2."
-      effort="10"
-      velocity="1" />
-  </joint>
-  <link
-    name="link_5">
-    <inertial>
-      <origin
-        xyz="0.0157361252272143 -0.00262703094861139 2.63403024947095E-08"
-        rpy="0 0 0" />
-      <mass
-        value="0.085015418080232" />
-      <inertia
-        ixx="3.37375916928367E-05"
-        ixy="7.89636338140576E-07"
-        ixz="4.15346591669036E-09"
-        iyy="2.0351585706133E-05"
-        iyz="-6.77065399053462E-08"
-        izz="2.66047123656453E-05" />
-    </inertial>
-    <visual>
-      <origin
-        xyz="0 0 0"
-        rpy="0 0 0" />
-      <geometry>
-        <mesh
-          filename="file:///home/ri-one/Open-Manipulator-X-6/complete_arm_assembly/urdf/../meshes/link_5.STL" />
-      </geometry>
-      <material
-        name="">
-        <color
-          rgba="0.894117647058823 0.894117647058823 0.894117647058823 1" />
-      </material>
-    </visual>
-    <collision>
-      <origin
-        xyz="0 0 0"
-        rpy="0 0 0" />
-      <geometry>
-        <mesh
-          filename="file:///home/ri-one/Open-Manipulator-X-6/complete_arm_assembly/urdf/../meshes/link_5.STL" />
-      </geometry>
-    </collision>
-  </link>
-  <joint
-    name="joint_5"
-    type="revolute">
-    <origin
-      xyz="0.086402 0.02425 0.0005"
-      rpy="0.036324 0 0" />
-    <parent
-      link="link_4" />
-    <child
-      link="link_5" />
-    <axis
-      xyz="1 0 0" />
-    <limit
-      lower="-3.14"
-      upper="3.14"
-      effort="10"
-      velocity="1" />
-  </joint>
-  <link
-    name="left_finger">
-    <inertial>
-      <origin
-        xyz="-0.019263 -1.6285 -1.7856"
-        rpy="0 0 0" />
-      <mass
-        value="0.0274218714255595" />
-      <inertia
-        ixx="7.35775440757057E-06"
-        ixy="3.29947226227772E-09"
-        ixz="-2.17679083297117E-07"
-        iyy="8.21755225888586E-06"
-        iyz="-1.77060574885703E-10"
-        izz="1.30421803809744E-05" />
-    </inertial>
-    <visual>
-      <origin
-        xyz="0 0 0"
-        rpy="0 0 0" />
-      <geometry>
-        <mesh
-          filename="file:///home/ri-one/Open-Manipulator-X-6/complete_arm_assembly/urdf/../meshes/left_finger.STL" />
-      </geometry>
-      <material
-        name="">
-        <color
-          rgba="0.894117647058823 0.894117647058823 0.894117647058823 1" />
-      </material>
-    </visual>
-    <collision>
-      <origin
-        xyz="0 0 0"
-        rpy="0 0 0" />
-      <geometry>
-        <mesh
-          filename="file:///home/ri-one/Open-Manipulator-X-6/complete_arm_assembly/urdf/../meshes/left_finger.STL" />
-      </geometry>
-    </collision>
-  </link>
-  <joint
-    name="left_finger_joint"
-    type="prismatic">
-    <origin
-      xyz="-0.019263 -1.6285 -1.7856"
-      rpy="0 0 0" />
-    <parent
-      link="link_5" />
-    <child
-      link="left_finger" />
-    <axis
-      xyz="0 0 1" />
-    <limit
-      lower="0"
-      upper="0.019"
-      effort="5"
-      velocity="0.1" />
-  </joint>
-  <link
-    name="right_finger">
-    <inertial>
-      <origin
-        xyz="-0.0408496815010922 1.72245379516032 2.02780677437668"
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