Commit message: Updated limits for joint 4

File: complete_arm_assembly/urdf/complete_arm_assembly_urdf.xacro (robot description, xacro)
@@ -272,6 +272,6 @@
       xyz="0 0 1" />
     <limit
-      lower="-1.8"
-      upper="1.8"
+      lower="-1"
+      upper="2.6"
       effort="10"
       velocity="1" />

File: complete_arm_assembly/urdf/fixed.urdf (robot description, URDF)
Before this commit: robot complete_arm_assembly, 8 links, 7 joints
Joints:
- joint joint_4: limit lower=-1.8 upper=1.8 effort=10 velocity=1 -> lower=-1 upper=2.6 effort=10 velocity=1

Commit message: Added the world_to_base_joint

File: complete_arm_assembly/urdf/complete_arm_assembly_urdf.xacro (robot description, xacro)
@@ -455,3 +455,9 @@
       offset="0" />
   </joint>
+  <link name="world"/>
+  <joint name="world_to_base_joint" type="fixed">
+    <parent link="world"/>
+    <child link="base_link"/>
+    <origin xyz="0 0 0" rpy="0 0 0"/>
+  </joint>
 </robot>

File: complete_arm_assembly/urdf/fixed.urdf (robot description, URDF)
Before this commit: robot complete_arm_assembly, 8 links, 7 joints
Links:
- added link world
Joints:
- added joint world_to_base_joint: type fixed, parent world, child base_link, origin xyz=0 0 0 rpy=0 0 0
- joint joint_4: limit lower=-1 upper=2.6 effort=10 velocity=1 -> lower=-1 upper=2. effort=10 velocity=1

Commit message: Update joint limits for left and right fingers

File: complete_arm_assembly/urdf/complete_arm_assembly_urdf.xacro (robot description, xacro)
@@ -194,5 +194,5 @@
     <child link="left_finger" />
     <axis xyz="0 0 1" />
-    <limit lower="0" upper="0.019" effort="5" velocity="0.1" />
+    <limit lower="0" upper="0.019" effort="20" velocity="0.2" />
     <dynamics damping="50.0" friction="5.0"/>
   </joint>
@@ -228,5 +228,5 @@
     <child link="right_finger" />
     <axis xyz="0 0 -1" />
-    <limit lower="-0.019" upper="0.0" effort="5" velocity="0.1" />
+    <limit lower="-0.019" upper="0.0" effort="20" velocity="0.2" />
     <dynamics damping="50.0" friction="5.0"/>
   </joint>

Commit message: Configured Gazebo environment

File: complete_arm_assembly/urdf/complete_arm_assembly_urdf.xacro (robot description, xacro)
@@ -153,5 +153,4 @@
     </collision>
   </link>
-  <!-- joint_5 damping increased to stabilize wrist carrying finger loads -->
   <joint name="joint_5" type="revolute">
     <origin xyz="0.086402 0.02425 0.0005" rpy="0.036324 0 0" />
@@ -166,8 +165,4 @@
       <origin xyz="0 0 0" rpy="0 0 0" />
       <mass value="0.05" />
-      <!-- Parallel axis theorem: joint origin is ~1.63m in Y, ~1.79m in Z from link_5
-           ixx = 0.0001 + 0.05*(1.6285^2 + 1.7856^2) = 0.292
-           iyy = 0.0001 + 0.05*(0.019^2  + 1.7856^2) = 0.159
-           izz = 0.0001 + 0.05*(0.019^2  + 1.6285^2) = 0.133 -->
       <inertia ixx="0.292" ixy="0" ixz="0"
                            iyy="0.159" iyz="0"
@@ -188,5 +183,4 @@
     </collision>
   </link>
-  <!-- Finger joint damping massively increased to suppress oscillation from large lever arm -->
   <joint name="left_finger_joint" type="prismatic">
     <origin xyz="-0.019263 -1.6285 -1.7856" rpy="0 0 0" />
@@ -194,5 +188,5 @@
     <child link="left_finger" />
     <axis xyz="0 0 1" />
-    <limit lower="0" upper="0.019" effort="20" velocity="0.2" />
+    <limit lower="0" upper="0.019" effort="5" velocity="0.1" />
     <dynamics damping="50.0" friction="5.0"/>
   </joint>
@@ -201,8 +195,4 @@
       <origin xyz="0 0 0" rpy="0 0 0" />
       <mass value="0.05" />
-      <!-- Parallel axis theorem: joint origin is ~1.61m in Y, ~1.79m in Z from link_5
-           ixx = 0.0001 + 0.05*(1.6058^2 + 1.7856^2) = 0.288
-           iyy = 0.0001 + 0.05*(0.019^2  + 1.7856^2) = 0.159
-           izz = 0.0001 + 0.05*(0.019^2  + 1.6058^2) = 0.129 -->
       <inertia ixx="0.288" ixy="0" ixz="0"
                            iyy="0.159" iyz="0"
@@ -228,5 +218,5 @@
     <child link="right_finger" />
     <axis xyz="0 0 -1" />
-    <limit lower="-0.019" upper="0.0" effort="20" velocity="0.2" />
+    <limit lower="-0.019" upper="0.0" effort="5" velocity="0.1" />
     <dynamics damping="50.0" friction="5.0"/>
   </joint>
