Commit message: Update mesh file paths to lowercase

File: URDF/end_effector_full_build/urdf/End Effector Full Build.urdf (robot description, URDF)
Before this commit: robot End Effector Full Build, 4 links, 3 joints
Links:
- link base_link: geometry collision mesh filename=package://end_effector_full_build/meshes/base_link.STL; visual mesh filename=package://end_effector_full_build/meshes/base_link.STL
- link finger_1: geometry collision mesh filename=package://end_effector_full_build/meshes/finger_1.STL; visual mesh filename=package://end_effector_full_build/meshes/finger_1.STL
- link finger_2: geometry collision mesh filename=package://end_effector_full_build/meshes/finger_2.STL; visual mesh filename=package://end_effector_full_build/meshes/finger_2.STL
- link ring_link: geometry collision mesh filename=package://end_effector_full_build/meshes/ring_link.STL; visual mesh filename=package://end_effector_full_build/meshes/ring_link.STL
